File: updi_hv_reset.kicad_pcb (KiCad board)
At the start: 2 copper layers, 38 x 25 mm, 32 parts, among them J1 UPDI, J2 USB, J3 SW, Q1 DMG2301L, U1 CH340E, U2 NCP1529A, U3 MT3608

Commit message: README and pics added
Parts:
- C9: value 1n -> 10n
- J2: footprint Connector_PinHeader_2.54mm:PinHeader_1x04_P2.54mm_Vertical -> Connector_JST:JST_XH_B4B-XH-A_1x04_P2.50mm_Vertical
- LED2: value PWR -> PRG
- Q1: value DMG2301L -> PMV65XP
- moved J2 7.63 mm to (102.3, 116.2), turned to 90 degrees
Connections:
- J2 pad 1: GND -> +5V
- J2 pad 2: UDP -> UDM
- J2 pad 3: UDM -> UDP
- J2 pad 4: +5V -> GND
Changed lines of the file:
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@@
   (net 20 "unconnected-(U1-~{CTS}-Pad5)")
   (net 21 "unconnected-(U3-NC-Pad6)")
-  (footprint "Connector_PinHeader_2.54mm:PinHeader_1x04_P2.54mm_Vertical" (layer "F.Cu")
-    (at 102.19 108.57)
-    (descr "Through hole straight pin header, 1x04, 2.54mm pitch, single row")
-    (tags "Through hole pin header THT 1x04 2.54mm single row")
+  (footprint "Connector_JST:JST_XH_B4B-XH-A_1x04_P2.50mm_Vertical" (layer "F.Cu")
+    (at 102.27 116.2 90)
+    (descr "JST XH series connector, B4B-XH-A (http://www.jst-mfg.com/product/pdf/eng/eXH.pdf), generated with kicad-footprint-generator")
+    (tags "connector JST XH vertical")
     (property "Sheetfile" "updi_hv_reset.kicad_sch")
     (property "Sheetname" "")
@@
     (property "ki_keywords" "connector")
     (attr through_hole)
-    (fp_text reference "J2" (at 0.1 -2.81) (layer "F.SilkS")
-        (effects (font (size 1 1) (thickness 0.15)))
-    )
-    (fp_text value "USB" (at 0.03 10.55) (layer "F.SilkS")
-        (effects (font (size 1 1) (thickness 0.15)))
-    )
-    (fp_text user "${REFERENCE}" (at 0 3.81 90) (layer "F.Fab")
-        (effects (font (size 1 1) (thickness 0.15)))
-    )
-    (fp_line (start -1.33 -1.33) (end 0 -1.33)
-      (stroke (width 0.12) (type solid)) (layer "F.SilkS"))
-    (fp_line (start -1.33 0) (end -1.33 -1.33)
-      (stroke (width 0.12) (type solid)) (layer "F.SilkS"))
-    (fp_line (start -1.33 1.27) (end -1.33 8.95)
-      (stroke (width 0.12) (type solid)) (layer "F.SilkS"))
-    (fp_line (start -1.33 1.27) (end 1.33 1.27)
-      (stroke (width 0.12) (type solid)) (layer "F.SilkS"))
-    (fp_line (start -1.33 8.95) (end 1.33 8.95)
-      (stroke (width 0.12) (type solid)) (layer "F.SilkS"))
-    (fp_line (start 1.33 1.27) (end 1.33 8.95)
-      (stroke (width 0.12) (type solid)) (layer "F.SilkS"))
-    (fp_line (start -1.8 -1.8) (end -1.8 9.4)
-      (stroke (width 0.05) (type solid)) (layer "F.CrtYd"))
-    (fp_line (start -1.8 9.4) (end 1.8 9.4)
-      (stroke (width 0.05) (type solid)) (layer "F.CrtYd"))
-    (fp_line (start 1.8 -1.8) (end -1.8 -1.8)
-      (stroke (width 0.05) (type solid)) (layer "F.CrtYd"))
-    (fp_line (start 1.8 9.4) (end 1.8 -1.8)
-      (stroke (width 0.05) (type solid)) (layer "F.CrtYd"))
-    (fp_line (start -1.27 -0.635) (end -0.635 -1.27)
-      (stroke (width 0.1) (type solid)) (layer "F.Fab"))
-    (fp_line (start -1.27 8.89) (end -1.27 -0.635)
-      (stroke (width 0.1) (type solid)) (layer "F.Fab"))
-    (fp_line (start -0.635 -1.27) (end 1.27 -1.27)
-      (stroke (width 0.1) (type solid)) (layer "F.Fab"))
-    (fp_line (start 1.27 -1.27) (end 1.27 8.89)
-      (stroke (width 0.1) (type solid)) (layer "F.Fab"))
-    (fp_line (start 1.27 8.89) (end -1.27 8.89)
-      (stroke (width 0.1) (type solid)) (layer "F.Fab"))
-    (pad "1" thru_hole rect (at 0 0) (size 1.7 1.7) (drill 1) (layers "*.Cu" "*.Mask")
-      (net 2 "GND") (pinfunction "Pin_1") (pintype "passive"))
-    (pad "2" thru_hole oval (at 0 2.54) (size 1.7 1.7) (drill 1) (layers "*.Cu" "*.Mask")
-      (net 13 "UDP") (pinfunction "Pin_2") (pintype "passive"))
-    (pad "3" thru_hole oval (at 0 5.08) (size 1.7 1.7) (drill 1) (layers "*.Cu" "*.Mask")
-      (net 14 "UDM") (pinfunction "Pin_3") (pintype "passive"))
-    (pad "4" thru_hole oval (at 0 7.62) (size 1.7 1.7) (drill 1) (layers "*.Cu" "*.Mask")
-      (net 3 "+5V") (pinfunction "Pin_4") (pintype "passive"))
-    (model "${KICAD6_3DMODEL_DIR}/Connector_PinHeader_2.54mm.3dshapes/PinHeader_1x04_P2.54mm_Vertical.wrl"
+    (fp_text reference "J2" (at 11.12 0.25 180) (layer "F.SilkS")
+        (effects (font (size 1 1) (thickness 0.15)))
+    )
+    (fp_text value "USB" (at -3.81 0.14 180) (layer "F.Fab")
+        (effects (font (size 1 1) (thickness 0.15)))
+    )
+    (fp_text user "${REFERENCE}" (at 3.75 2.7 90) (layer "F.Fab")
+        (effects (font (size 1 1) (thickness 0.15)))
+    )
+    (fp_line (start -2.85 -2.75) (end -2.85 -1.5)
+      (stroke (width 0.12) (type solid)) (layer "F.SilkS"))
+    (fp_line (start -2.56 -2.46) (end -2.56 3.51)
+      (stroke (width 0.12) (type solid)) (layer "F.SilkS"))
+    (fp_line (start -2.56 3.51) (end 10.06 3.51)
+      (stroke (width 0.12) (type solid)) (layer "F.SilkS"))
+    (fp_line (start -2.55 -2.45) (end -2.55 -1.7)
+      (stroke (width 0.12) (type solid)) (layer "F.SilkS"))
+    (fp_line (start -2.55 -1.7) (end -0.75 -1.7)
+      (stroke (width 0.12) (type solid)) (layer "F.SilkS"))
+    (fp_line (start -2.55 -0.2) (end -1.8 -0.2)
+      (stroke (width 0.12) (type solid)) (layer "F.SilkS"))
+    (fp_line (start -1.8 -0.2) (end -1.8 2.75)
+      (stroke (width 0.12) (type solid)) (layer "F.SilkS"))
+    (fp_line (start -1.8 2.75) (end 3.75 2.75)
+      (stroke (width 0.12) (type solid)) (layer "F.SilkS"))
+    (fp_line (start -1.6 -2.75) (end -2.85 -2.75)
+      (stroke (width 0.12) (type solid)) (layer "F.SilkS"))
+    (fp_line (start -0.75 -2.45) (end -2.55 -2.45)
+      (stroke (width 0.12) (type solid)) (layer "F.SilkS"))
+    (fp_line (start -0.75 -1.7) (end -0.75 -2.45)
+      (stroke (width 0.12) (type solid)) (layer "F.SilkS"))
+    (fp_line (start 0.75 -2.45) (end 0.75 -1.7)
+      (stroke (width 0.12) (type solid)) (layer "F.SilkS"))
+    (fp_line (start 0.75 -1.7) (end 6.75 -1.7)
+      (stroke (width 0.12) (type solid)) (layer "F.SilkS"))
+    (fp_line (start 6.75 -2.45) (end 0.75 -2.45)
+      (stroke (width 0.12) (type solid)) (layer "F.SilkS"))
+    (fp_line (start 6.75 -1.7) (end 6.75 -2.45)
+      (stroke (width 0.12) (type solid)) (layer "F.SilkS"))
+    (fp_line (start 8.25 -2.45) (end 8.25 -1.7)
+      (stroke (width 0.12) (type solid)) (layer "F.SilkS"))
+    (fp_line (start 8.25 -1.7) (end 10.05 -1.7)
+      (stroke (width 0.12) (type solid)) (layer "F.SilkS"))
+    (fp_line (start 9.3 -0.2) (end 9.3 2.75)
+      (stroke (width 0.12) (type solid)) (layer "F.SilkS"))
+    (fp_line (start 9.3 2.75) (end 3.75 2.75)
+      (stroke (width 0.12) (type solid)) (layer "F.SilkS"))
+    (fp_line (start 10.05 -2.45) (end 8.25 -2.45)
+      (stroke (width 0.12) (type solid)) (layer "F.SilkS"))
+    (fp_line (start 10.05 -1.7) (end 10.05 -2.45)
+      (stroke (width 0.12) (type solid)) (layer "F.SilkS"))
+    (fp_line (start 10.05 -0.2) (end 9.3 -0.2)
+      (stroke (width 0.12) (type solid)) (layer "F.SilkS"))
+    (fp_line (start 10.06 -2.46) (end -2.56 -2.46)
+      (stroke (width 0.12) (type solid)) (layer "F.SilkS"))
+    (fp_line (start 10.06 3.51) (end 10.06 -2.46)
+      (stroke (width 0.12) (type solid)) (layer "F.SilkS"))
+    (fp_line (start -2.95 -2.85) (end -2.95 3.9)
+      (stroke (width 0.05) (type solid)) (layer "F.CrtYd"))
+    (fp_line (start -2.95 3.9) (end 10.45 3.9)
+      (stroke (width 0.05) (type solid)) (layer "F.CrtYd"))
+    (fp_line (start 10.45 -2.85) (end -2.95 -2.85)
+      (stroke (width 0.05) (type solid)) (layer "F.CrtYd"))
+    (fp_line (start 10.45 3.9) (end 10.45 -2.85)
+      (stroke (width 0.05) (type solid)) (layer "F.CrtYd"))
+    (fp_line (start -2.45 -2.35) (end -2.45 3.4)
+      (stroke (width 0.1) (type solid)) (layer "F.Fab"))
+    (fp_line (start -2.45 3.4) (end 9.95 3.4)
+      (stroke (width 0.1) (type solid)) (layer "F.Fab"))
+    (fp_line (start -0.625 -2.35) (end 0 -1.35)
+      (stroke (width 0.1) (type solid)) (layer "F.Fab"))
+    (fp_line (start 0 -1.35) (end 0.625 -2.35)
+      (stroke (width 0.1) (type solid)) (layer "F.Fab"))
+    (fp_line (start 9.95 -2.35) (end -2.45 -2.35)
+      (stroke (width 0.1) (type solid)) (layer "F.Fab"))
+    (fp_line (start 9.95 3.4) (end 9.95 -2.35)
+      (stroke (width 0.1) (type solid)) (layer "F.Fab"))
+    (pad "1" thru_hole oval (at 0 0 90) (size 1.7 1.95) (drill 0.95) (layers "*.Cu" "*.Mask")
+      (net 3 "+5V") (pinfunction "Pin_1") (pintype "passive"))
+    (pad "2" thru_hole oval (at 2.5 0 90) (size 1.7 1.95) (drill 0.95) (layers "*.Cu" "*.Mask")
+      (net 14 "UDM") (pinfunction "Pin_2") (pintype "passive"))
+    (pad "3" thru_hole oval (at 5 0 90) (size 1.7 1.95) (drill 0.95) (layers "*.Cu" "*.Mask")
+      (net 13 "UDP") (pinfunction "Pin_3") (pintype "passive"))
+    (pad "4" thru_hole roundrect (at 7.5 0 90) (size 1.7 1.95) (drill 0.95) (layers "*.Cu" "*.Mask") (roundrect_rratio 0.25)
+      (net 2 "GND") (pinfunction "Pin_4") (pintype "passive"))
+    (model "${KICAD6_3DMODEL_DIR}/Connector_JST.3dshapes/JST_XH_B4B-XH-A_1x04_P2.50mm_Vertical.wrl"
       (offset (xyz 0 0 0))
       (scale (xyz 1 1 1))
@@
     (property "ki_keywords" "cap capacitor")
     (attr smd)
-    (fp_text reference "C1" (at 0 -1.85 90) (layer "F.SilkS")
+    (fp_text reference "C1" (at 3.34 -0.05 90) (layer "F.SilkS")
         (effects (font (size 1 1) (thickness 0.15)))
     )
@@
         (effects (font (size 1 1) (thickness 0.15)))
     )
-    (fp_text value "PWR" (at 0 1.65) (layer "F.Fab")
+    (fp_text value "PRG" (at 0 1.65) (layer "F.Fab")
         (effects (font (size 1 1) (thickness 0.15)))
     )
@@
         (effects (font (size 1 1) (thickness 0.15)) (justify mirror))
     )
-    (fp_text value "1n" (at 0 -1.85) (layer "B.Fab")
+    (fp_text value "10n" (at 0 -1.85) (layer "B.Fab")
         (effects (font (size 1 1) (thickness 0.15)) (justify mirror))
     )
@@
         (effects (font (size 1 1) (thickness 0.15)) (justify mirror))
     )
-    (fp_text value "DMG2301L" (at 0 -2.4) (layer "B.Fab")
-        (effects (font (size 1 1) (thickness 0.15)) (justify mirror))
-    )
+    (fp_text value "PMV65XP" (at 0 -2.4) (layer "B.Fab")
+        (effects (font (size 1 1) (thickness 0.15)) (justify mirror))
+    )
