File: updi_hv_reset.kicad_sch (KiCad schematic)
At the start: 32 parts, among them J1 UPDI, J2 USB, J3 SW, Q1 PMV65XP, U1 CH340E, U2 NCP1529A, U3 MT3608

Commit message: README and pics added
Parts:
- J2: footprint Connector_PinHeader_2.54mm:PinHeader_1x04_P2.54mm_Vertical -> Connector_JST:JST_XH_B4B-XH-A_1x04_P2.50mm_Vertical
- LED2: value PWR -> PRG
Connections:
- net +5V: now also J2.1 (Pin_1); no longer J2.4 (Pin_4)
- net GND: now also J2.4 (Pin_4); no longer J2.1 (Pin_1)
- net UDM: now also J2.2 (Pin_2); no longer J2.3 (Pin_3)
- net UDP: now also J2.3 (Pin_3); no longer J2.2 (Pin_2)
Other:
- company: (none) -> SGGDEV
- title: (none) -> UPDI_HV_PROGRAMMER_ILYA2IK
- moved on the sheet: C9, J2, J3, L1
